Commit message: add bumper

File: g13_description/urdf/g13.gazebo.xacro (robot description, xacro)
@@ -5,5 +5,5 @@
   <xacro:arg name="imu_visual"    default="false"/>
   <gazebo reference="base_link">
-    <material>Gazebo/Yellow</material>
+    <!-- <material>Gazebo/Yellow</material> -->
     <material>Gazebo/${player_color}</material>
   </gazebo>
@@ -169,3 +169,16 @@
     </sensor>
   </gazebo>
+  <gazebo reference="base_link">
+    <sensor name="base_link" type="contact">
+      <update_rate>1000.0</update_rate>
+      <always_on>true</always_on>
+      <contact>
+        <collision> base_footprint_fixed_joint_lump__base_link_collision </collision>
+      </contact>
+      <plugin name="base_link_contact_sensor_plugin" filename="libgazebo_ros_bumper.so">
+        <bumperTopicName>contact</bumperTopicName>
+        <frameName>world</frameName>
+      </plugin>
+    </sensor>
+  </gazebo>
 </robot>
