Commit message: add proper mesh

File: g12_description/urdf/g12.urdf.xacro (robot description, xacro)
@@ -23,5 +23,4 @@
         <mesh filename="package://turtlebot3_description/meshes/bases/waffle_pi_base.stl" scale="0.001 0.001 0.001"/>
       </geometry>
-<!--      <material name="light_black"/>-->
       <material name="$(arg player_color)"/>
     </visual>
@@ -193,5 +192,5 @@
     <visual>
       <geometry>
-        <box size="0.015 0.030 0.027" />
+        <mesh filename="package://g12_description/meshes/kinect_camera_simple.stl" scale="1.0 1.0 1.0"/>
       </geometry>
     </visual>

Commit message: Driver now ocntrols joint

File: g12_description/urdf/g12.urdf.xacro (robot description, xacro)
@@ -44,4 +44,5 @@
     <origin xyz="0.0 0.144 0.023" rpy="-1.57 0 0"/>
     <axis xyz="0 0 1"/>
+    <limit effort="30" velocity="0.3" />
   </joint>
   <link name="wheel_left_link">

Commit message: reduced camera rot speed

File: g12_description/urdf/g12.urdf.xacro (robot description, xacro)
@@ -174,4 +174,5 @@
     <child link="camera_link"/>
     <axis xyz="0 0 1"/>
+    <limit effort="30" velocity="0.3" />
   </joint>
   <link name="camera_link">
