Commit message: Continuous camera added

File: g12_description/urdf/g12.gazebo.xacro (robot description, xacro)
@@ -136,4 +136,18 @@
     </sensor>
   </gazebo>
+  <gazebo>
+    <plugin name="gazebo_ros_control" filename="libgazebo_ros_control.so">
+      <robotNamespace>/red1</robotNamespace>
+    </plugin>
+  </gazebo>
+  <transmission name="tran2">
+    <type>transmission_interface/SimpleTransmission</type>
+    <joint name="camera_joint">
+      <hardwareInterface>hardware_interface/EffortJointInterface</hardwareInterface>
+    </joint>
+    <actuator name="motor1">
+      <mechanicalReduction>1</mechanicalReduction>
+    </actuator>
+  </transmission>
   <!--link : https://www.raspberrypi.org/documentation/hardware/camera/-->
   <!-- <gazebo reference="camera_rgb_frame">

File: g12_description/urdf/g12.urdf.xacro (robot description, xacro)
@@ -170,17 +170,30 @@
     </inertial>
   </link>
-  <joint name="camera_joint" type="fixed">
+  <joint name="camera_joint" type="continuous">
 <!--    <origin xyz="0.073 -0.011 0.084" rpy="0 0 0"/>-->
     <origin xyz="0.073 -0.011 0.584" rpy="0 0.45 0"/>
     <parent link="base_link"/>
     <child link="camera_link"/>
+    <axis xyz="0 0 1"/>
   </joint>
   <link name="camera_link">
-    <collision>
-      <origin xyz="0.005 0.011 0.013" rpy="0 0 0"/>
-      <geometry>
+    <origin xyz="0.005 0.011 0.013" rpy="0.0 0.0 0.0"/>
+    <collision>
+      <geometry>
+        <cylinder length="0.0315" radius="0.055"/>
         <box size="0.015 0.030 0.027"/>
       </geometry>
     </collision>
+    <inertial>
+      <mass value="0.114" />
+      <inertia ixx="0.001" ixy="0.0" ixz="0.0"
+               iyy="0.001" iyz="0.0"
+               izz="0.001" />
+    </inertial>
+    <visual>
+      <geometry>
+        <box size="0.015 0.030 0.027" />
+      </geometry>
+    </visual>
   </link>
   <joint name="camera_rgb_joint" type="fixed">

Commit message: Fix joint motion

File: g12_description/urdf/g12.gazebo.xacro (robot description, xacro)
@@ -136,18 +136,4 @@
     </sensor>
   </gazebo>
-  <gazebo>
-    <plugin name="gazebo_ros_control" filename="libgazebo_ros_control.so">
-      <robotNamespace>/red1</robotNamespace>
-    </plugin>
-  </gazebo>
-  <transmission name="tran2">
-    <type>transmission_interface/SimpleTransmission</type>
-    <joint name="camera_joint">
-      <hardwareInterface>hardware_interface/EffortJointInterface</hardwareInterface>
-    </joint>
-    <actuator name="motor1">
-      <mechanicalReduction>1</mechanicalReduction>
-    </actuator>
-  </transmission>
   <!--link : https://www.raspberrypi.org/documentation/hardware/camera/-->
   <!-- <gazebo reference="camera_rgb_frame">
@@ -233,3 +219,18 @@
     </sensor>
   </gazebo>
+  <gazebo>
+  <plugin name="gazebo_ros_control" filename="libgazebo_ros_control.so">
+    <robotNamespace>/${player_name}</robotNamespace>
+  </plugin>
+</gazebo>
+<transmission name="tran1">
+    <type>transmission_interface/SimpleTransmission</type>
+    <joint name="camera_joint">
+      <hardwareInterface>hardware_interface/EffortJointInterface</hardwareInterface>
+    </joint>
+    <actuator name="motor1">
+      <hardwareInterface>EffortJointInterface</hardwareInterface>
+      <mechanicalReduction>1</mechanicalReduction>
+    </actuator>
+  </transmission>
 </robot>

File: g12_description/urdf/g12.urdf.xacro (robot description, xacro)
@@ -34,5 +34,4 @@
       <origin xyz="0 0 0" rpy="0 0 0"/>
       <mass value="1.3729096e+00"/>
-<!--      <mass value="100.3729096e+00"/>-->
       <inertia ixx="8.7002718e-03" ixy="-4.7576583e-05" ixz="1.1160499e-04"
                iyy="8.6195418e-03" iyz="-3.5422299e-06"
@@ -170,6 +169,5 @@
   </link>
   <joint name="camera_joint" type="continuous">
-<!--    <origin xyz="0.073 -0.011 0.084" rpy="0 0 0"/>-->
-    <origin xyz="0.073 -0.011 0.584" rpy="0 0.45 0"/>
+    <origin xyz="-0.1 0.0 0.3" rpy="0 0 0"/>
     <parent link="base_link"/>
     <child link="camera_link"/>
@@ -177,22 +175,22 @@
   </joint>
   <link name="camera_link">
-    <origin xyz="0.005 0.011 0.013" rpy="0.0 0.0 0.0"/>
-    <collision>
-      <geometry>
-        <cylinder length="0.0315" radius="0.055"/>
-        <box size="0.015 0.030 0.027"/>
-      </geometry>
-    </collision>
-    <inertial>
-      <mass value="0.114" />
-      <inertia ixx="0.001" ixy="0.0" ixz="0.0"
-               iyy="0.001" iyz="0.0"
-               izz="0.001" />
-    </inertial>
-    <visual>
+    <collision>
+      <origin xyz="0.005 0.011 0.013" rpy="0 0 0"/>
       <geometry>
         <mesh filename="package://g12_description/meshes/kinect_camera_simple.stl" scale="1.0 1.0 1.0"/>
       </geometry>
-    </visual>
+    </collision>
+    <visual>
+      <geometry>
+        <mesh filename="package://g12_description/meshes/kinect_camera_simple.stl" scale="1.0 1.0 1.0"/>
+      </geometry>
+    </visual>
+    <inertial>
+      <origin xyz="0.0 0.0 0.0" rpy="0 0 0"/>
+      <mass value="0.001" />
+      <inertia ixx="0.001" ixy="0.0" ixz="0.0"
+               iyy="0.001" iyz="0.0"
+               izz="0.001" />
+    </inertial>
   </link>
   <joint name="camera_rgb_joint" type="fixed">

Commit message: update kienct color

File: g12_description/urdf/g12.gazebo.xacro (robot description, xacro)
@@ -5,5 +5,4 @@
   <xacro:arg name="imu_visual"    default="false"/>
   <gazebo reference="base_link">
-    <!-- <material>Gazebo/Yellow</material> -->
     <material>Gazebo/${player_color}</material>
   </gazebo>
@@ -169,4 +168,5 @@
   </gazebo> -->
   <gazebo reference="camera_link">
+    <material>Gazebo/${player_color}</material>
     <sensor name="camera_link_camera" type="depth">
       <update_rate>3.0</update_rate>

Commit message: update camera pose

File: g12_description/urdf/g12.gazebo.xacro (robot description, xacro)
@@ -172,5 +172,5 @@
       <update_rate>3.0</update_rate>
       <camera>
-        <horizontal_fov>2.085595</horizontal_fov>
+        <horizontal_fov>1.047198</horizontal_fov>
         <image>
           <width>640</width>
@@ -190,5 +190,5 @@
         <pointCloudTopicName>depth/points</pointCloudTopicName>
         <frameName>camera_rgb_optical_frame</frameName>
-        <pointCloudCutoff>0.5</pointCloudCutoff>
+        <pointCloudCutoff>0.2</pointCloudCutoff>
         <pointCloudCutoffMax>3.0</pointCloudCutoffMax>
         <distortionK1>0.00000001</distortionK1>

File: g12_description/urdf/g12.urdf.xacro (robot description, xacro)
@@ -170,13 +170,19 @@
   </link>
   <joint name="camera_joint" type="continuous">
-    <origin xyz="-0.1 0.0 0.3" rpy="0 0 0"/>
-    <parent link="base_link"/>
-    <child link="camera_link"/>
+    <origin xyz="-0.05 0.0 0.35" rpy="0 0 0"/>
+    <parent link="base_link"/>
+    <child link="camera_link_aux"/>
     <axis xyz="0 0 1"/>
     <limit effort="30" velocity="0.3" />
   </joint>
+  <link name="camera_link_aux"/>
+  <joint name="camera_joint_aux" type="fixed">
+    <origin xyz="0.0 0.0 0.0" rpy="0 0.4 0"/>
+    <parent link="camera_link_aux"/>
+    <child link="camera_link"/>
+  </joint>
   <link name="camera_link">
     <collision>
-      <origin xyz="0.005 0.011 0.013" rpy="0 0 0"/>
+      <origin xyz="0.0 0.0 0.0" rpy="0 0 0"/>
       <geometry>
         <mesh filename="package://g12_description/meshes/kinect_camera_simple.stl" scale="1.0 1.0 1.0"/>

Commit message: Added wall ignore and revert camera changes

File: g12_description/urdf/g12.gazebo.xacro (robot description, xacro)
@@ -172,5 +172,5 @@
       <update_rate>3.0</update_rate>
       <camera>
-        <horizontal_fov>1.047198</horizontal_fov>
+        <horizontal_fov>2.085595</horizontal_fov>
         <image>
           <width>640</width>
@@ -190,5 +190,5 @@
         <pointCloudTopicName>depth/points</pointCloudTopicName>
         <frameName>camera_rgb_optical_frame</frameName>
-        <pointCloudCutoff>0.2</pointCloudCutoff>
+        <pointCloudCutoff>0.5</pointCloudCutoff>
         <pointCloudCutoffMax>3.0</pointCloudCutoffMax>
         <distortionK1>0.00000001</distortionK1>

File: g12_description/urdf/g12.urdf.xacro (robot description, xacro)
@@ -170,19 +170,12 @@
   </link>
   <joint name="camera_joint" type="continuous">
-    <origin xyz="-0.05 0.0 0.35" rpy="0 0 0"/>
-    <parent link="base_link"/>
-    <child link="camera_link_aux"/>
+    <origin xyz="-0.1 0.0 0.3" rpy="0 0 0"/>
+    <parent link="base_link"/>
+    <child link="camera_link"/>
     <axis xyz="0 0 1"/>
-    <limit effort="30" velocity="0.3" />
-  </joint>
-  <link name="camera_link_aux"/>
-  <joint name="camera_joint_aux" type="fixed">
-    <origin xyz="0.0 0.0 0.0" rpy="0 0.4 0"/>
-    <parent link="camera_link_aux"/>
-    <child link="camera_link"/>
   </joint>
   <link name="camera_link">
     <collision>
-      <origin xyz="0.0 0.0 0.0" rpy="0 0 0"/>
+      <origin xyz="0.005 0.011 0.013" rpy="0 0 0"/>
       <geometry>
         <mesh filename="package://g12_description/meshes/kinect_camera_simple.stl" scale="1.0 1.0 1.0"/>
